File: Braille-Column-Rods-PCB/Braille_Cell_Column.kicad_sch (KiCad schematic)
At the start: 11 parts, among them M6 Stepper_Motor_bipolar, U22 MT910xET, U7 DRV8847SPWR

Commit message: Polish prep for Rev 2 release, PCBA work
Parts:
- R27: value 2k1 -> 5k1
- U22: value MT910xET -> MT9101ET; LCSC (none) -> C2977713
Changed lines of the file:
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@@
 	(title_block
 		(title "Braille Cam Rod Prototype (Type 4)")
-		(date "2025-01-06")
-		(rev "Rev 1")
+		(date "2025-02-03")
+		(rev "Rev 2")
 	)
 	(junction
@@
 			)
 		)
-		(property "Value" "2k1"
+		(property "Value" "5k1"
 			(at 54.61 102.8699 0)
 			(effects
@@
 			)
 		)
-		(property "Value" "MT910xET"
+		(property "Value" "MT9101ET"
 			(at 125.73 43.1799 0)
 			(effects
@@
 			(at 129.54 41.91 0)
 			(effects
+				(font
+					(size 1.27 1.27)
+				)
+				(hide yes)
+			)
+		)
+		(property "LCSC" "C2977713"
+			(at 129.54 41.91 0)
+			(effects

Commit message: chore: bump to KiCAD v8 on re-save
Parts:
- renumbered C6 to C1, C22 to C17, C30 to C25, D9 to D1, M6 to M1, R26 to R1, R27 to R5, R28 to R6, R29 to R7, U7 to U1, U22 to U17

Commit message: feat: add INA219 current sensor
Parts:
- D1: value LED -> RED_LED
Changed lines of the file:
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@@
 			)
 		)
-		(property "Value" "LED"
+		(property "Value" "RED_LED"
 			(at 55.88 115.8874 90)
 			(effects
