File: Braille-Column-Rods-PCB/Microcontroller.kicad_sch (KiCad schematic)
At the start: 9 parts, among them J3 Conn_01x02, J4 Conn_01x08, SW1 SW_Push, SW2 SW_Push, U3 RP2040-Zero

Commit message: Polish prep for Rev 2 release, PCBA work
Parts:
- removed SW1, SW2: SW_Push, 00-lib-footprints:PushButtonSMD_2.93x3.9, symbol Switch:SW_Push
- added SW1, SW2: Tactile Button, 160gf, PCM_JLCPCB:SW-SMD_4P-L5.1-W5.1-P3.70-LS6.5-TL-2, symbol PCM_JLCPCB-Connectors_Buttons:Tactile Button, 160gf
- U3: symbol 00-project-symbols:RP2040-Zero -> 00-lib-symbols:RP2040-Zero; Source (none) -> https://github.com/dj505/RP2040-Zero-KiCAD
Connections:
- net GND: now also SW1.3 (C), SW1.4 (D), SW2.3 (C), SW2.4 (D)
- net SW_1: now also SW1.1 (A), SW1.2 (B)
- net SW_2: now also SW2.1 (A), SW2.2 (B)
