File: Braille-Column-Rods-PCB/Motor_Control.kicad_sch (KiCad schematic)
At the start: 7 parts, among them U14 74HC595, U15 74HC595, U30 CD74HC4067M

Commit message: Polish prep for Rev 2 release, PCBA work
Parts:
- added R42, R44, R45: 5k1, Resistor_SMD:R_0603_1608Metric_Pad0.98x0.95mm_HandSolder, symbol Device:R
- U14, U15: LCSC (none) -> C5947
Connections:
- net +3V3: now also R42.1
- net GND: now also R44.2, R45.2
- net at U30.16 (I15): now also R45.1
- net ANALOG_DEMO_1: now reaches U30.17 (I14)
- net ANALOG_DEMO_1: now also R42.2, R44.1
- no-connect marks 13 -> 11

Commit message: feat: add INA219 current sensor
Other:
- note added: "Hall Sensor Switch"
- note removed: "Hall Effect Switch"
Changed lines of the file:
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@@
 		)
 	)
-	(text "Hall Effect Switch"
+	(text "Hall Sensor Switch"
 		(exclude_from_sim no)
 		(at 227.33 57.404 0)
